Commit message: urdf changes, zennoh helper scrits

File: ros2_ws/src/project_bringup/urdf/phoenix.urdf (robot description, URDF)
Before this commit: robot phoenix_slam, 2 links, 1 joints
Links:
- link base_link: geometry collision mesh filename=package://robot_model/meshes/model.stl scale=0.005 0.005 0.005; visual mesh filename=package://robot_model/meshes/model.stl scale=0.005 0.005 0.005
